Commit message: fix: размер колеи

File: ijkbot_description/urdf/ijkbot.urdf.xacro (robot description, xacro)
@@ -4,5 +4,5 @@
   <xacro:property name="wheel_radius" value="0.0375"/>  <!-- D = 75 мм -->
   <xacro:property name="wheel_width" value="0.025"/>
-  <xacro:property name="wheel_separation" value="0.225"/> <!-- L = 225 мм, колея по центрам -->
+  <xacro:property name="wheel_separation" value="0.225"/> <!-- L = 225 мм -->
   <xacro:property name="wheel_offset_y" value="${wheel_separation / 2.0}"/>
   <xacro:property name="chassis_length" value="0.220"/>

Commit message: feat(bringup): единый мастер-лаунч system.launch.py для одновременного запуска робота и Nav2

File: ijkbot_description/urdf/ijkbot.urdf.xacro (robot description, xacro)
@@ -111,9 +111,14 @@
     <origin xyz="${caster_offset_x} -${caster_offset_y} ${-wheel_radius + 0.015}" rpy="0 0 0"/>
   </joint>
+  <!-- Параметры установки камеры Intel RealSense D435 -->
+  <xacro:property name="camera_offset_x" value="0.05"/>
+  <xacro:property name="camera_offset_y" value="0.0"/>
+  <xacro:property name="camera_offset_z" value="0.12"/>
+  <xacro:property name="camera_pitch" value="0.0"/>   <!-- Наклон камеры (рад). 0.0 = строго параллельно полу -->
   <!-- Крепление камеры Intel RealSense D435 -->
   <joint name="camera_joint" type="fixed">
     <parent link="base_link"/>
     <child link="camera_link"/>
-    <origin xyz="0.05 0 0.12" rpy="0 0 0"/>
+    <origin xyz="${camera_offset_x} ${camera_offset_y} ${camera_offset_z}" rpy="0 ${camera_pitch} 0"/>
   </joint>
   <link name="camera_link">
